Commit message: am

File: 3DOF/model/link_dimensions.xacro (robot description, xacro)
@@ -3,6 +3,6 @@
     <!-- Constants -->
     <xacro:property name="LENGTH" value="1.0"/>
-    <xacro:property name="WIDTH" value="0.1"/>
-    <xacro:property name="HEIGHT" value="0.1"/>
-    <xacro:property name="RADIUS" value="${WIDTH / 2.0}"/>
+    <xacro:property name="WIDTH" value="0.05"/>
+    <xacro:property name="HEIGHT" value="0.05"/>
+    <xacro:property name="RADIUS" value="0.05"/>
 </robot>

File: 3DOF/model/model.urdf (robot description, URDF)
Before this commit: robot manipulator, 5 links, 4 joints
Links:
- link base_link: geometry collision box size=0.05 0.05 0.05; visual box size=0.05 0.05 0.05
- link cylinder1: geometry collision cylinder length=0.05 radius=0.05; visual cylinder length=0.05 radius=0.05
- link cylinder2: geometry collision cylinder length=0.05 radius=0.05; visual cylinder length=0.05 radius=0.05
- link link1: geometry collision box size=1.0 0.05 0.05; visual box size=1.0 0.05 0.05
- link link2: geometry collision box size=1.0 0.05 0.05; visual box size=1.0 0.05 0.05
Joints:
- joint joint1: origin xyz=0.1 0 0 rpy=0.0 0.0 0.0 -> xyz=0.05 0 0 rpy=0.0 0.0 0.0
- joint joint2: origin xyz=0.1 0 0 rpy=0.0 0.0 0.0 -> xyz=0.05 0 0 rpy=0.0 0.0 0.0

File: 3DOF/model/model.xacro (robot description, xacro)
@@ -1,6 +1,9 @@
 <?xml version="1.0"?>
 <robot name="manipulator" xmlns:xacro="http://www.ros.org/wiki/xacro">
+<xacro:include filename="$(find 3DOF)/model/transmissions.xacro" />
+<xacro:include filename="$(find 3DOF)/model/manipulator.gazebo" />
 <xacro:include filename="$(find 3DOF)/model/link_dimensions.xacro" />
 <xacro:include filename="$(find 3DOF)/model/physics.xacro" />
+<xacro:include filename="$(find pr2_description)/urdf/sensors/hokuyo_lx30_laser.urdf.xacro" />
 <link name="base_link">
     <visual>
@@ -62,5 +65,5 @@
 		<parent link="cylinder1"/>
 		<child link="link1"/>
-		<origin rpy="0.0 0.0 0.0" xyz="${2.0 * RADIUS} 0 0"/>
+		<origin rpy="0.0 0.0 0.0" xyz="${RADIUS} 0 0"/>
 		<limit effort="${effort}" velocity="${velocity}" lower="${lower_bound}" upper="${upper_bound}"/>
                 <dynamics damping="${damping}" />
@@ -126,5 +129,5 @@
 		<parent link="cylinder2"/>
 		<child link="link2"/>
-		<origin rpy="0.0 0.0 0.0" xyz="${2.0 * RADIUS} 0 0"/>
+		<origin rpy="0.0 0.0 0.0" xyz="${RADIUS} 0 0"/>
 		<limit effort="${effort}" velocity="${velocity}" lower="${lower_bound}" upper="${upper_bound}"/>
                 <dynamics damping="${damping}" />
@@ -154,99 +157,7 @@
                 </inertial>
 </link>
-<!--<joint name="joint2" type="revolute">
-		<axis xyz="0 0 1"/>
-		<parent link="cylinder2"/>
-		<child link="link2"/>
-		<origin rpy="0.0 0.0 0.0" xyz="0.01 0 0"/>
-		<limit effort="${effort}" velocity="${velocity}" lower="${lower_bound}" upper="${upper_bound}"/>
-                <dynamics damping="${damping}" />
-</joint>
-<link name="link2">
-		<visual>
-			<origin rpy="0.0 0.0 0.0" xyz="${0.01 + (LENGTH / 2.0)} 0 0"/>
-			<geometry>
-			        <box size="${LENGTH} ${WIDTH} ${HEIGHT}" />
-			</geometry>
-			<material name="green">
-				<color rgba="0 .8 0 1"/>
-			</material>
-		</visual>
-		<collision>
-			<origin rpy="0.0 0.0 0.0" xyz="${0.01 + (LENGTH / 2.0)} 0 0"/>
-			<geometry>
-				<box size="${LENGTH} ${WIDTH} ${HEIGHT}" />
-			</geometry>
-		</collision>
-                <inertial>
-                        <origin xyz="0 0 0" rpy="0 0 0"/>
-                        <mass value="${coxa_mass}" />
-                        <inertia ixx="${ixx}" ixy="${ixy}" ixz="${ixz}"
-                 iyy="${iyy}" iyz="${iyz}"
-                 izz="${izz}" />
-                </inertial>
-</link>
-<joint name="joint2" type="revolute">
-		<axis xyz="0 0 1"/>
-		<parent link="link1"/>
-		<child link="link2"/>
-		<origin rpy="0.0 0.0 0.0" xyz="${LENGTH} 0 0"/>
-		<limit effort="${effort}" velocity="${velocity}" lower="${lower_bound}" upper="${upper_bound}"/>
-                <dynamics damping="${damping}" />
-</joint>
-<link name="link2">
-		<visual>
-			<origin rpy="0.0 0.0 0.0" xyz="${LENGTH / 2.0} 0 0"/>
-			<geometry>
-				<box size="${LENGTH} ${WIDTH} ${HEIGHT}" />
-			</geometry>
-			<material name="blue">
-				<color rgba="0 0 .8 1"/>
-			</material>
-		</visual>
-		<collision>
-			<origin rpy="0.0 0.0 0.0" xyz="${LENGTH / 2.0} 0 0"/>
-			<geometry>
-				<box size="${LENGTH} ${WIDTH} ${HEIGHT}" />
-			</geometry>
-		</collision>
-                <inertial>
-                        <origin xyz="0 0 0" rpy="0 0 0"/>
-                        <mass value="${coxa_mass}" />
-                        <inertia ixx="${ixx}" ixy="${ixy}" ixz="${ixz}"
-                 iyy="${iyy}" iyz="${iyz}"
-                 izz="${izz}" />
-                </inertial>
-</link>
-<joint name="joint3" type="revolute">
-		<axis xyz="0 0 1"/>
-		<parent link="link2"/>
-		<child link="link3"/>
-		<origin rpy="0.0 0.0 0.0" xyz="${LENGTH} 0 0"/>
-		<limit effort="${effort}" velocity="${velocity}" lower="${lower_bound}" upper="${upper_bound}"/>
-                <dynamics damping="${damping}" />
-</joint>
-<link name="link3">
-		<visual>
-			<origin rpy="0.0 0.0 0.0" xyz="${LENGTH / 2.0} 0 0"/>
-			<geometry>
-				<box size="${LENGTH} ${WIDTH} ${HEIGHT}" />
-			</geometry>
-			<material name="red">
-				<color rgba="0.8 0 0 1"/>
-			</material>
-		</visual>
-		<collision>
-			<origin rpy="0.0 0.0 0.0" xyz="${LENGTH / 2.0} 0 0"/>
-			<geometry>
-				<box size="${LENGTH} ${WIDTH} ${HEIGHT}" />
-			</geometry>
-		</collision>
-                <inertial>
-                        <origin xyz="0 0 0" rpy="0 0 0"/>
-                        <mass value="${coxa_mass}" />
-                        <inertia ixx="${ixx}" ixy="${ixy}" ixz="${ixz}"
-                 iyy="${iyy}" iyz="${iyz}"
-                 izz="${izz}" />
-                </inertial>
-</link>-->
+<!--<xacro:hokuyo_lx30_laser_v0 name="side_laser" parent="link2" ros_topic="side_scan"
+                            update_rate="20" min_angle="-1.57" max_angle="1.57" >
+                            <origin xyz="0 -.220 0.200" rpy="0 0 0" />
+</xacro:hokuyo_lx30_laser_v0>-->
 </robot>
